File: Teleschtroumpf_PCB/Teleschtroumpf.kicad_pcb (KiCad board)
At the start: 2 copper layers, 85 x 48 mm, 9 parts, among them IC1 ESP32-DEVKITC-VE, Q2 BC337

Commit message: PCB Update (better ESP32 footprint)
Parts:
- removed IC1: ESP32-DEVKITC-VE, KiCad:ESP32DEVKITCVE
- added U1: ESP32-S3-DevKitC-1-N32R16V, LIB_ESP32-S3-DevKitC-1-N32R16V:ESP32S3DevKitC1N32R16V, F.Cu at (121.1, 63.0)
- moved R1 11.0 mm to (79.4, 55.0)
- moved Q2 9.88 mm to (130.0, 82.5), turned to -90 degrees
- moved R2 7.38 mm to (130.0, 62.9)
- moved LA1 1.12 mm to (124.1, 55.0)
Routing:
- net Net-(LA1-+): track 26.3 -> 14.3 mm
- net Net-(U1-16): track 39.3 -> 32.9 mm
- net Net-(LA1--): track 41.0 -> 35.5 mm
- net Net-(Q2-B): track 9.46 -> 7.55 mm
- net Net-(U1-5V): track 11.2 -> 12.4 mm
Other:
- board text added: "Téléschtroumpf"
