File: Teleschtroumpf_PCB/Teleschtroumpf.kicad_sch (KiCad schematic)
At the start: 9 parts, among them IC1 ESP32-DEVKITC-VE, Q2 BC337

Commit message: PCB Update (better ESP32 footprint)
Parts:
- removed IC1: ESP32-DEVKITC-VE, KiCad:ESP32DEVKITCVE, symbol ESP32-DEVKITC-VE:ESP32-DEVKITC-VE
- added U1: ESP32-S3-DevKitC-1-N32R16V, LIB_ESP32-S3-DevKitC-1-N32R16V:ESP32S3DevKitC1N32R16V, symbol ESP32-S3-DevKitC-1-N32R16V:ESP32-S3-DevKitC-1-N32R16V
Connections:
- net at R1.1: now also U1.J131 (5V)
- net at R2.1: now also U1.J119 (16)
- net at Q2.3 (E): now also U1.J311 (G_2)
Other:
- moved on the sheet: R1
